File: v1/dediprog_interface/spi_dediprog_interface.kicad_pcb (KiCad board)
At the start: 2 copper layers, 20 x 27 mm, 3 parts, among them J1 Conn_02x10_Odd_Even, J2 Conn_01x02_Pin, J4 Conn_01x10_Socket

Commit message: WIP: Redesign
Parts:
- removed J2: Conn_01x02_Pin, Connector_PinHeader_2.54mm:PinHeader_1x02_P2.54mm_Vertical
- added D1: LED, LED_SMD:LED_0805_2012Metric, F.Cu at (12.7, 29.7)
- added J3: Conn_01x02_Pin, Connector_PinHeader_2.54mm:PinHeader_1x02_P2.54mm_Vertical, F.Cu at (17.4, 21.6)
- added R1: R100, Resistor_SMD:R_0805_2012Metric, F.Cu at (8.80, 24.0)
- added R2: R300, Resistor_SMD:R_0805_2012Metric, F.Cu at (8.78, 26.3)
- added SW1: SW_Push, Button_Switch_SMD:SW_Tactile_SPST_NO_Straight_CK_PTS636Sx25SMTRLFS, F.Cu at (17.1, 29.6)
- added U1: ~, Package_DIP:SMDIP-4_W7.62mm, F.Cu at (5.40, 31.6)
- J1: moved to B.Cu
- J4: moved to F.Cu
- moved J1 2.56 mm to (2.21, 2.60), turned to 180 degrees
- moved J4 2.22 mm to (15.1, 9.50), turned to 90 degrees
Connections:
- J4 pad 1: GND -> Net-(J4-Pin_1)
- J4 pad 10: Net-(J2-Pin_1) -> GND
- J4 pad 2: +3.3V -> P_IO3
- J4 pad 3: P_CS1 -> P_IO2
- J4 pad 4: P_CS2 -> P_MISO
- J4 pad 5: P_CLK -> P_MOSI
- J4 pad 6: P_MOSI -> P_CLK
- J4 pad 7: P_MISO -> P_CS2
- J4 pad 8: P_IO2 -> P_CS1
- J4 pad 9: P_IO3 -> +3.3V
Routing:
- net Net-(J4-Pin_1): track 0.00 -> 32.4 mm
- net GND: track 26.3 -> 51.7 mm
- net Net-(J3-Pin_1): track 0.00 -> 25.1 mm
- net +3.3V: track 10.5 -> 23.2 mm
- net Net-(J2-Pin_1): track 12.7 -> 0.00 mm
- net Net-(R1-Pad2): track 0.00 -> 11.9 mm
- net Net-(J3-Pin_2): track 0.00 -> 10.3 mm
- net P_CS1: track 7.37 -> 16.0 mm
- net P_CS2: track 18.9 -> 10.7 mm
- net P_IO2: track 7.34 -> 14.6 mm
- net P_MISO: track 7.98 -> 12.6 mm, vias 0 -> 1
- net P_IO3: track 15.1 -> 19.6 mm, vias 0 -> 1
- net Net-(D1-A): track 0.00 -> 4.05 mm
- net P_CLK: track 12.9 -> 9.01 mm
- net P_MOSI: track 12.8 -> 9.72 mm, vias 1 -> 0
- added copper zone on B.Cu, net GND
- added copper zone on F.Cu, net GND
Other:
- board size 20 x 27 mm -> 20 x 34.7 mm
- board text added: "GND"
- board text added: "RST"
