File: v1/spi_implant/SPI_Implant.kicad_pcb (KiCad board)
At the start: 2 copper layers, 25.9 x 18.9 mm, 14 parts, among them J1 Conn_01x10_Socket, J2 SPI_Socket, J3 Conn_01x01, U1 TMUX1511PWR, U2 TMUX1511PWR

Commit message: WIP: Redesign
Parts:
- moved C1 6.44 mm to (9.00, 17.4), turned to 180 degrees
- moved R1 4.76 mm to (9.00, 6.40)
- moved R5 4.64 mm to (9.00, 8.60)
- moved R4 4.52 mm to (8.97, 10.8)
- moved R3 4.41 mm to (9.00, 13.0)
- moved R2 4.30 mm to (9.00, 15.2)
- moved U1 4.03 mm to (14.1, 4.25), turned to -90 degrees
- moved C2 3.98 mm to (8.90, 1.30)
- moved D1 3.55 mm to (9.00, 3.90)
- moved J3 2.90 mm to (18.6, 1.40)
- moved U2 2.26 mm to (14.1, 14.6), turned to -90 degrees
Routing:
- net +3.3V: track 47.5 -> 70.1 mm, vias 2 -> 6
- net P_MOSI: track 20.7 -> 5.74 mm, vias 2 -> 0
- net CLK: track 14.1 -> 2.54 mm, vias 2 -> 0
- net P_IO3: track 19.0 -> 10.5 mm
- net IO2: track 13.2 -> 5.40 mm
- net CS1: track 8.27 -> 16.0 mm
- net IO3: track 3.20 -> 10.7 mm
- net CS2: track 8.24 -> 15.3 mm, vias 0 -> 2
- net MISO: track 14.9 -> 8.85 mm, vias 2 -> 0
- net Net-(J2-Pin_5): track 2.71 -> 7.61 mm
- net Net-(J2-Pin_6): track 2.71 -> 7.53 mm
- net Net-(J2-Pin_7): track 2.67 -> 7.43 mm
- net Net-(J2-Pin_8): track 2.69 -> 7.38 mm
- net Net-(J2-Pin_9): track 2.69 -> 7.30 mm
- net P_CS1: track 18.0 -> 13.9 mm
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Other:
- board text added: "RST"
- board text removed: "reset"
