File: v1/spi_implant/SPI_Implant.kicad_sch (KiCad schematic)
At the start: 13 parts, among them J1 Conn_01x10_Socket, J2 SPI_Socket, J3 Conn_01x01, U1 TMUX1511PWR, U2 TMUX1511PWR

Commit message: WIP: Redesign
Parts:
- added D2, D3, D4: WS2812B, LED_SMD:LED_WS2812B_PLCC4_5.0x5.0mm_P3.2mm, symbol LED:WS2812B
